File: headstageNano.sch (EAGLE design)
At the start: 8 parts, among them U1 RHD2132_QFN

Commit message: ungrounded pin 33 elec_test for impedance tests
Connections:
- net GND: no longer U1.ELEC_TEST
Changed lines of the file:
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@@
 <part name="C_REF" library="resistor" deviceset="C-US" device="C0402K" value="0.1uF"/>
 <part name="GND1" library="supply1" deviceset="GND" device=""/>
-<part name="GND2" library="supply1" deviceset="GND" device=""/>
 <part name="VDD1" library="supply1" deviceset="VDD" device=""/>
 <part name="VDD2" library="supply1" deviceset="VDD" device=""/>
@@
 <instance part="C_REF" gate="G$1" x="43.18" y="-33.02" rot="R90"/>
 <instance part="GND1" gate="1" x="45.72" y="-2.54" rot="R90"/>
-<instance part="GND2" gate="1" x="40.64" y="0" rot="R90"/>
 <instance part="VDD1" gate="G$1" x="53.34" y="-7.62" rot="R270"/>
 <instance part="VDD2" gate="G$1" x="40.64" y="-66.04" rot="R270"/>
@@
 </segment>
 <segment>
-<pinref part="U1" gate="A" pin="ELEC_TEST"/>
-<wire x1="33.02" y1="0" x2="38.1" y2="0" width="0.1524" layer="91"/>
-<pinref part="GND2" gate="1" pin="GND"/>
-</segment>
-<segment>

Commit message: updating capacitor values
Parts:
- C_REF: value 0.1uF -> 10 nF
- C_VDD: value 10uF -> 100 nF
Changed lines of the file:
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@@
 <part name="R2" library="resistor" deviceset="R-EU_" device="R0402" value="100"/>
 <part name="R3" library="resistor" deviceset="R-EU_" device="R0402" value="100"/>
-<part name="C_VDD" library="resistor" deviceset="C-US" device="C0402K" value="10uF"/>
-<part name="C_REF" library="resistor" deviceset="C-US" device="C0402K" value="0.1uF"/>
+<part name="C_VDD" library="resistor" deviceset="C-US" device="C0402K" value="100 nF"/>
+<part name="C_REF" library="resistor" deviceset="C-US" device="C0402K" value="10 nF"/>
 <part name="GND1" library="supply1" deviceset="GND" device=""/>
 <part name="VDD1" library="supply1" deviceset="VDD" device=""/>
